Commit message: ROS: Valter URDF (exps)

File: software/ROS/models/valter/urdf/valter/robots/valter.URDF (robot description, URDF)
Before this commit: robot valter, 3 links, 2 joints
Links:
- added link support_wheels, mass 1.30791131979034; collision mesh filename=package://valter/meshes/support_wheels.STL; visual mesh filename=package://valter/meshes/support_wheels.STL
- added link support_wheels_centers, mass 0.101015328916835; collision mesh filename=package://valter/meshes/support_wheels_centers.STL; visual mesh filename=package://valter/meshes/support_wheels_centers.STL
- link Base: mass 40 -> 12.6713271850958
- link LWheel: mass 2 -> 3.69869087372323
- link RWheel: mass 2 -> 3.69869087372323
Joints:
- added joint support_wheels_centers_fixed: type fixed, parent support_wheels, child support_wheels_centers, origin xyz=0 0 -0.22244 rpy=0 0 0, axis 0 0 0
- added joint support_wheels_fixed: type fixed, parent Base, child support_wheels, origin xyz=0.18923 -0.1113 0.067926 rpy=1.5708 0 0, axis 0 0 0
- joint RWheelAxis: limit (none) -> effort=0 velocity=0

Commit message: ROS: Valter URDF model (in pregress, learning)

File: software/ROS/models/valter/urdf/valter/robots/valter.URDF (robot description, URDF)
Before this commit: robot valter, 5 links, 4 joints
Links:
- added link ManipulatorBase, mass 0.17883; collision mesh filename=package://valter/meshes/ManipulatorBase.STL; visual mesh filename=package://valter/meshes/ManipulatorBase.STL
- added link ManipulatorLink1, mass 4; collision mesh filename=package://valter/meshes/ManipulatorLink1.STL; visual mesh filename=package://valter/meshes/ManipulatorLink1.STL
- added link ManipulatorLink2, mass 2; collision mesh filename=package://valter/meshes/ManipulatorLink2.STL; visual mesh filename=package://valter/meshes/ManipulatorLink2.STL
- added link ManipulatorLink3, mass 0.22788; collision mesh filename=package://valter/meshes/ManipulatorLink3.STL; visual mesh filename=package://valter/meshes/ManipulatorLink3.STL
- added link lwheel_centers, mass 0.0783773140784395; collision mesh filename=package://valter/meshes/lwheel_centers.STL; visual mesh filename=package://valter/meshes/lwheel_centers.STL
- added link rwheel_centers, mass 0.0783773140784392; collision mesh filename=package://valter/meshes/rwheel_centers.STL; visual mesh filename=package://valter/meshes/rwheel_centers.STL
- link Base: mass 12.6713271850958 -> 12.623
- link LWheel: mass 3.69869087372323 -> 3.6203
- link RWheel: mass 3.69869087372323 -> 3.6203
- link support_wheels: mass 1.30791131979034 -> 1.3079
Joints:
- added joint ManipulatorBaseFixed: type fixed, parent Base, child ManipulatorBase, origin xyz=0.157269945428792 0.0354609509421621 0.707041900761443 rpy=1.5707963267949 0 3.14159265358979, axis 0 0 0
- added joint ManipulatorLink1Axis: type revolute, parent ManipulatorBase, child ManipulatorLink1, origin xyz=0.015824 -0.0090419 0 rpy=3.1416 0 3.1416, axis 0 0 -1, limit lower=-1 upper=0 effort=0 velocity=0
- added joint ManipulatorLink2Axis: type revolute, parent ManipulatorLink1, child ManipulatorLink2, origin xyz=0.10656 -0.49054 0 rpy=0 0 0, axis 0 0 -1, limit lower=0 upper=1 effort=0 velocity=0
- added joint ManipulatorLink3Axis: type revolute, parent ManipulatorLink2, child ManipulatorLink3, origin xyz=-0.012962 0.55415 0 rpy=0 0 0, axis 0 0 -1, limit lower=-0.5 upper=1 effort=0 velocity=0
- added joint lwheel_centers_fixed: type fixed, parent LWheel, child lwheel_centers, origin xyz=0 -0.00181724367610836 0 rpy=0 -1.66371525153719E-34 0, axis 0 1 0
- added joint rwheel_centers_fixed: type fixed, parent RWheel, child rwheel_centers, origin xyz=0 -0.00181724367610836 0 rpy=3.14159265358979 0 0, axis 0 1 0
- joint LWheelAxis: origin xyz=0.00034158 0.15432 0.14 rpy=6.6286E-17 0.39309 -3.1416 -> xyz=0.000341577688738742 0.154324334429763 0.14 rpy=6.6286088844449E-17 0.39309481042652 -3.14159265358979
- joint RWheelAxis: limit effort=0 velocity=0 -> (none); origin xyz=0.00034158 -0.15368 0.14 rpy=-6.123E-17 0 0 -> xyz=0.000341577688738742 -0.153675665570238 0.14 rpy=-6.12303176911189E-17 0 0
- joint support_wheels_centers_fixed: origin xyz=0 0 -0.22244 rpy=0 0 0 -> xyz=0 0 -0.222438597166117 rpy=0 0 0
- joint support_wheels_fixed: origin xyz=0.18923 -0.1113 0.067926 rpy=1.5708 0 0 -> xyz=0.189234607270609 -0.11129709785824 0.0679256801186866 rpy=1.5707963267949 0 0

Commit message: ROS: Valter URDF model (in progress)

File: software/ROS/models/valter/urdf/valter/robots/valter.URDF (robot description, URDF)
Before this commit: robot valter, 11 links, 10 joints
Links:
- added link GripperL, mass 0.039858; collision mesh filename=package://valter/meshes/GripperL.STL; visual mesh filename=package://valter/meshes/GripperL.STL
- added link GripperR, mass 0.039858; collision mesh filename=package://valter/meshes/GripperR.STL; visual mesh filename=package://valter/meshes/GripperR.STL
- added link ManipulatorLink4, mass 0.42935; collision mesh filename=package://valter/meshes/ManipulatorLink4.STL; visual mesh filename=package://valter/meshes/ManipulatorLink4.STL
- link Base: mass 12.623 -> 12.6233325032135
- link LWheel: mass 3.6203 -> 3.62031355964479
- link ManipulatorBase: mass 0.17883 -> 0.178834143520891
- link ManipulatorLink1: mass 4 -> 0.47801
- link ManipulatorLink2: mass 2 -> 0.30452
- link RWheel: mass 3.6203 -> 3.62031355964479
- link support_wheels: mass 1.3079 -> 1.30791131979034
Joints:
- added joint GripperLAxis: type prismatic, parent ManipulatorLink4, child GripperL, origin xyz=0.049892 0.090686 -0.0096825 rpy=3.1416 -6.9389E-17 -3.1416, axis -1 0 0, limit lower=-0.03 upper=0 effort=0 velocity=0
- added joint GripperRAxis: type prismatic, parent ManipulatorLink4, child GripperR, origin xyz=-0.049892 0.090686 -0.0096825 rpy=-4.9087E-21 6.9389E-17 1.0613E-16, axis 1 0 0, limit lower=0 upper=0.03 effort=0 velocity=0
- added joint ManipulatorLink4Axis: type revolute, parent ManipulatorLink3, child ManipulatorLink4, origin xyz=0 0.008 0.034995 rpy=0 1.5708 0, axis 0 -1 0, limit lower=-3 upper=3 effort=0 velocity=0
- joint ManipulatorLink1Axis: limit lower=-1 upper=0 effort=0 velocity=0 -> lower=-1.5 upper=0 effort=0 velocity=0
- joint ManipulatorLink2Axis: limit lower=0 upper=1 effort=0 velocity=0 -> lower=0 upper=1.5 effort=0 velocity=0
- joint ManipulatorLink3Axis: limit lower=-0.5 upper=1 effort=0 velocity=0 -> lower=0 upper=1 effort=0 velocity=0

Commit message: ROS: Valter's URDF model (preliminary done)

File: software/ROS/models/valter/urdf/valter/robots/valter.URDF (robot description, URDF)
Before this commit: robot valter, 14 links, 13 joints
Links:
- added link Head, mass 5.04298545454377; collision mesh filename=package://valter/meshes/Head.STL; visual mesh filename=package://valter/meshes/Head.STL
- added link LArm, mass 0.244790015736888; collision mesh filename=package://valter/meshes/LArm.STL; visual mesh filename=package://valter/meshes/LArm.STL
- added link LArmElbow, mass 0.0397123450849927; collision mesh filename=package://valter/meshes/LArmElbow.STL; visual mesh filename=package://valter/meshes/LArmElbow.STL
- added link LFinger0, mass 0.02336143148626; collision mesh filename=package://valter/meshes/LFinger0.STL; visual mesh filename=package://valter/meshes/LFinger0.STL
- added link LFinger1, mass 0.02336143148626; collision mesh filename=package://valter/meshes/LFinger1.STL; visual mesh filename=package://valter/meshes/LFinger1.STL
- added link LFinger2, mass 0.02336143148626; collision mesh filename=package://valter/meshes/LFinger2.STL; visual mesh filename=package://valter/meshes/LFinger2.STL
- added link LFinger3, mass 0.02336143148626; collision mesh filename=package://valter/meshes/LFinger3.STL; visual mesh filename=package://valter/meshes/LFinger3.STL
- added link LFinger4, mass 0.02336143148626; collision mesh filename=package://valter/meshes/LFinger4.STL; visual mesh filename=package://valter/meshes/LFinger4.STL
- added link LFinger5, mass 0.02336143148626; collision mesh filename=package://valter/meshes/LFinger5.STL; visual mesh filename=package://valter/meshes/LFinger5.STL
- added link LForearmRoll, mass 0.93501476271025; collision mesh filename=package://valter/meshes/LForearmRoll.STL; visual mesh filename=package://valter/meshes/LForearmRoll.STL
- added link LForearmYaw, mass 0.60265; collision mesh filename=package://valter/meshes/LForearmYaw.STL; visual mesh filename=package://valter/meshes/LForearmYaw.STL
- added link LHandPitch, mass 0.0061941814843542; collision mesh filename=package://valter/meshes/LHandPitch.STL; visual mesh filename=package://valter/meshes/LHandPitch.STL
- added link LHandYaw, mass 0.312277803709901; collision mesh filename=package://valter/meshes/LHandYaw.STL; visual mesh filename=package://valter/meshes/LHandYaw.STL
- added link LShoulder, mass 0.175328671502516; collision mesh filename=package://valter/meshes/LShoulder.STL; visual mesh filename=package://valter/meshes/LShoulder.STL
- added link LTorso, mass 7.0955682087774; collision mesh filename=package://valter/meshes/LTorso.STL; visual mesh filename=package://valter/meshes/LTorso.STL
- added link Neck, mass 0.264426936484469; collision mesh filename=package://valter/meshes/Neck.STL; visual mesh filename=package://valter/meshes/Neck.STL
- added link RArm, mass 0.244790015736889; collision mesh filename=package://valter/meshes/RArm.STL; visual mesh filename=package://valter/meshes/RArm.STL
- added link RArmElbow, mass 0.0397123450849928; collision mesh filename=package://valter/meshes/RArmElbow.STL; visual mesh filename=package://valter/meshes/RArmElbow.STL
- added link RFinger0, mass 0.02336143148626; collision mesh filename=package://valter/meshes/RFinger0.STL; visual mesh filename=package://valter/meshes/RFinger0.STL
- added link RFinger1, mass 0.02336143148626; collision mesh filename=package://valter/meshes/RFinger1.STL; visual mesh filename=package://valter/meshes/RFinger1.STL
- added link RFinger2, mass 0.02336143148626; collision mesh filename=package://valter/meshes/RFinger2.STL; visual mesh filename=package://valter/meshes/RFinger2.STL
- added link RFinger3, mass 0.02336143148626; collision mesh filename=package://valter/meshes/RFinger3.STL; visual mesh filename=package://valter/meshes/RFinger3.STL
- added link RFinger4, mass 0.02336143148626; collision mesh filename=package://valter/meshes/RFinger4.STL; visual mesh filename=package://valter/meshes/RFinger4.STL
- added link RFinger5, mass 0.0233614314862599; collision mesh filename=package://valter/meshes/RFinger5.STL; visual mesh filename=package://valter/meshes/RFinger5.STL
- added link RForearmRoll, mass 0.935014762710249; collision mesh filename=package://valter/meshes/RForearmRoll.STL; visual mesh filename=package://valter/meshes/RForearmRoll.STL
- added link RForearmYaw, mass 0.60265; collision mesh filename=package://valter/meshes/RForearmYaw.STL; visual mesh filename=package://valter/meshes/RForearmYaw.STL
- added link RHandPitch, mass 0.00619418148435421; collision mesh filename=package://valter/meshes/RHandPitch.STL; visual mesh filename=package://valter/meshes/RHandPitch.STL
- added link RHandYaw, mass 0.312277803709901; collision mesh filename=package://valter/meshes/RHandYaw.STL; visual mesh filename=package://valter/meshes/RHandYaw.STL
- added link RShoulder, mass 0.175328671502516; collision mesh filename=package://valter/meshes/RShoulder.STL; visual mesh filename=package://valter/meshes/RShoulder.STL
- added link RTorso, mass 7.0955682087774; collision mesh filename=package://valter/meshes/RTorso.STL; visual mesh filename=package://valter/meshes/RTorso.STL
- added link Torso, mass 12.3493829426964; collision mesh filename=package://valter/meshes/Torso.STL; visual mesh filename=package://valter/meshes/Torso.STL
- added link Trunk, mass 27.438; collision mesh filename=package://valter/meshes/Trunk.STL; visual mesh filename=package://valter/meshes/Trunk.STL
- link Base: mass 12.6233325032135 -> 12.7723641606721
- link GripperL: mass 0.039858 -> 0.0398581317877607
- link GripperR: mass 0.039858 -> 0.0398581317877607
- link ManipulatorLink1: mass 0.47801 -> 0.478012742893284
- link ManipulatorLink2: mass 0.30452 -> 0.304515245459477
- link ManipulatorLink3: mass 0.22788 -> 0.227882111375496
- link ManipulatorLink4: mass 0.42935 -> 0.42934890554545
Joints:
- removed joint GripperLAxis
- removed joint GripperRAxis
- removed joint LWheelAxis
- removed joint ManipulatorLink1Axis
- removed joint ManipulatorLink2Axis
- removed joint ManipulatorLink3Axis
- removed joint ManipulatorLink4Axis
- removed joint RWheelAxis
- added joint GripperLJoint: type prismatic, parent ManipulatorLink4, child GripperL, origin xyz=0.049892 0.090686 -0.0096825 rpy=3.1416 -6.9389E-17 -3.1416, axis -1 0 0, limit lower=-0.03 upper=0 effort=0 velocity=0
- added joint GripperRJoint: type prismatic, parent ManipulatorLink4, child GripperR, origin xyz=-0.049892 0.090686 -0.0096825 rpy=-4.9087E-21 6.9389E-17 1.0613E-16, axis 1 0 0, limit lower=0 upper=0.03 effort=0 velocity=0
- added joint HeadJoint: type revolute, parent Neck, child Head, origin xyz=0.0085 0.05 0 rpy=0 0 0, axis 0 0 -1, limit lower=0 upper=0.85 effort=0 velocity=0
- added joint LArmElbowJoint: type revolute, parent LArm, child LArmElbow, origin xyz=0 -0.39975 0 rpy=-1.5708 0 1.5708, axis 0 0 -1, limit lower=-0.9 upper=0.9 effort=0 velocity=0
- added joint LArmJoint: type revolute, parent LShoulder, child LArm, origin xyz=0 0.116 0 rpy=-3.1416 0 1.5708, axis 0 0 -1, limit lower=-1.5 upper=0 effort=0 velocity=0
- added joint LFinger0Joint: type revolute, parent LHandYaw, child LFinger0, origin xyz=0.01463 0.0125 -0.025 rpy=3.1416 0 2.3562, axis 0 0 1, limit lower=0 upper=1 effort=0 velocity=0
- added joint LFinger1Joint: type revolute, parent LHandYaw, child LFinger1, origin xyz=0.08863 0.0135 -0.02375 rpy=0 0 0, axis 0 0 -1, limit lower=-1 upper=0 effort=0 velocity=0
- added joint LFinger2Joint: type revolute, parent LHandYaw, child LFinger2, origin xyz=0.08863 0.0135 -0.00125 rpy=0 0 0, axis 0 0 -1, limit lower=-1 upper=0 effort=0 velocity=0
- added joint LFinger3Joint: type revolute, parent LHandYaw, child LFinger3, origin xyz=0.08863 0.0135 0.00125 rpy=0 0 0, axis 0 0 -1, limit lower=-1 upper=0 effort=0 velocity=0
- added joint LFinger4Joint: type revolute, parent LHandYaw, child LFinger4, origin xyz=0.08863 0.0135 0.02375 rpy=0 0 0, axis 0 0 -1, limit lower=-1 upper=0 effort=0 velocity=0
- added joint LFinger5Joint: type revolute, parent LHandYaw, child LFinger5, origin xyz=0.01463 0.0125 0.025 rpy=3.1416 0 2.3562, axis 0 0 1, limit lower=0 upper=1 effort=0 velocity=0
- added joint LForearmRollJoint: type revolute, parent LForearmYaw, child LForearmRoll, origin xyz=0 -0.055 0.0395 rpy=0 1.5708 0, axis 1 0 0, limit lower=-3.7 upper=0 effort=0 velocity=0
- added joint LForearmYawJoint: type revolute, parent LArmElbow, child LForearmYaw, origin xyz=-0.036 0 0 rpy=1.5708 1.5708 0, axis 0 -1 0, limit lower=-0.1 upper=0.4 effort=0 velocity=0
- added joint LHandPitchJoint: type revolute, parent LForearmRoll, child LHandPitch, origin xyz=-0.23422 -0.005 0 rpy=0 1.5708 0, axis -1 0 0, limit lower=-0.3 upper=0.5 effort=0 velocity=0
- added joint LHandYawJoint: type revolute, parent LHandPitch, child LHandYaw, origin xyz=0.0002314 0 -0.015731 rpy=0 1.5708 0, axis 0 -1 0, limit lower=-0.5 upper=0.2 effort=0 velocity=0
- added joint LShoulderJoint: type revolute, parent LTorso, child LShoulder, origin xyz=0.1085 0.31956 0.067 rpy=1.5708 0 1.5708, axis 0 1 0, limit lower=-1.5 upper=0.5 effort=0 velocity=0
- added joint LTorsoJoint: type revolute, parent Torso, child LTorso, origin xyz=0.10841 0 -0.09 rpy=3.1416 0 -3.1416, axis 0 -1 0, limit lower=0 upper=0.85 effort=0 velocity=0
- added joint LWheelJoint: type continuous, parent Base, child LWheel, origin xyz=0.000341577688738742 0.154324334429763 0.14 rpy=6.6286088844449E-17 0.39309481042652 -3.14159265358979, axis 0 -1 0
- added joint ManipulatorLink1Joint: type revolute, parent ManipulatorBase, child ManipulatorLink1, origin xyz=0.015824 -0.0090419 0 rpy=3.1416 0 3.1416, axis 0 0 -1, limit lower=-1.5 upper=0 effort=0 velocity=0
- added joint ManipulatorLink2Joint: type revolute, parent ManipulatorLink1, child ManipulatorLink2, origin xyz=0.10656 -0.49054 0 rpy=0 0 0, axis 0 0 -1, limit lower=0 upper=1.5 effort=0 velocity=0
- added joint ManipulatorLink3Joint: type revolute, parent ManipulatorLink2, child ManipulatorLink3, origin xyz=-0.012962 0.55415 0 rpy=0 0 0, axis 0 0 -1, limit lower=0 upper=1 effort=0 velocity=0
- added joint ManipulatorLink4Joint: type revolute, parent ManipulatorLink3, child ManipulatorLink4, origin xyz=0 0.008 0.034995 rpy=0 1.5708 0, axis 0 -1 0, limit lower=-3 upper=3 effort=0 velocity=0
- added joint NeckJoint: type revolute, parent Torso, child Neck, origin xyz=-0.00017682 0.42056 0 rpy=0 0 0, axis 0 -1 0, limit lower=-1.57 upper=1.57 effort=0 velocity=0
- added joint RArmElbowJoint: type revolute, parent RArm, child RArmElbow, origin xyz=0 -0.39975 0 rpy=1.5708 8.6736E-16 1.5708, axis 0 0 -1, limit lower=-0.9 upper=0.9 effort=0 velocity=0
- added joint RArmJoint: type revolute, parent RShoulder, child RArm, origin xyz=0 0.116 0 rpy=-3.1416 1.3305E-19 1.5709, axis 0 0 1, limit lower=0 upper=1.5 effort=0 velocity=0
- added joint RFinger0Joint: type revolute, parent RHandYaw, child RFinger0, origin xyz=0.01463 0.0125 0.025 rpy=-3.1416 -3.3278E-08 2.3562, axis 0 0 1, limit lower=0 upper=1 effort=0 velocity=0
- added joint RFinger1Joint: type revolute, parent RHandYaw, child RFinger1, origin xyz=0.08863 0.0135 0.02375 rpy=1.4439E-11 9.4125E-08 0.0003068, axis 0 0 -1, limit lower=-1 upper=0 effort=0 velocity=0
- added joint RFinger2Joint: type revolute, parent RHandYaw, child RFinger2, origin xyz=0.08863 0.0135 0.00125 rpy=1.4439E-11 9.4125E-08 0.0003068, axis 0 0 -1, limit lower=-1 upper=0 effort=0 velocity=0
- added joint RFinger3Joint: type revolute, parent RHandYaw, child RFinger3, origin xyz=0.08863 0.0135 -0.00125 rpy=1.4439E-11 9.4125E-08 0.0003068, axis 0 0 -1, limit lower=-1 upper=0 effort=0 velocity=0
- added joint RFinger4Joint: type revolute, parent RHandYaw, child RFinger4, origin xyz=0.08863 0.0135 -0.02375 rpy=1.4439E-11 9.4125E-08 0.0003068, axis 0 0 -1, limit lower=-1 upper=0 effort=0 velocity=0
- added joint RFinger5Joint: type revolute, parent RHandYaw, child RFinger5, origin xyz=0.01463 0.0125 -0.025 rpy=-3.1416 -3.3278E-08 2.3562, axis 0 0 1, limit lower=0 upper=1 effort=0 velocity=0
- added joint RForearmRollJoint: type revolute, parent RForearmYaw, child RForearmRoll, origin xyz=0 -0.055013 0.0395 rpy=3.1414 1.5708 3.1416, axis 1 0 0, limit lower=0 upper=3.7 effort=0 velocity=0
- added joint RForearmYawJoint: type revolute, parent RArmElbow, child RForearmYaw, origin xyz=-0.035987 0 0 rpy=4.0616E-07 1.5708 -1.5708, axis 0 -1 0, limit lower=-0.4 upper=0.1 effort=0 velocity=0
- added joint RHandPitchJoint: type revolute, parent RForearmRoll, child RHandPitch, origin xyz=-0.23422 -0.005 0 rpy=-0.00030678 1.5708 1.9045E-08, axis -1 0 0, limit lower=-0.3 upper=0.5 effort=0 velocity=0
- added joint RHandYawJoint: type revolute, parent RHandPitch, child RHandYaw, origin xyz=0.0002314 0 -0.015731 rpy=3.1416 1.5708 3.1416, axis 0 -1 0, limit lower=-0.2 upper=0.5 effort=0 velocity=0
- added joint RShoulderJoint: type revolute, parent RTorso, child RShoulder, origin xyz=0.1085 0.31956 -0.067 rpy=-1.5708 0 1.5708, axis 0 -1 0, limit lower=-1.5 upper=0.5 effort=0 velocity=0
- added joint RTorsoJoint: type revolute, parent Torso, child RTorso, origin xyz=0.10841 0 0.09 rpy=3.1416 0 -3.1416, axis 0 -1 0, limit lower=-0.85 upper=0 effort=0 velocity=0
- added joint RWheelJoint: type continuous, parent Base, child RWheel, origin xyz=0.000341577688738742 -0.153675665570238 0.14 rpy=-6.12303176911189E-17 0 0, axis 0 1 0
- added joint TorsoJoint: type revolute, parent Trunk, child Torso, origin xyz=0 0.45 0 rpy=0 0 0, axis 0 0 -1, limit lower=0 upper=1 effort=0 velocity=0
- added joint TrunkJoint: type revolute, parent Base, child Trunk, origin xyz=-0.01423 0.00097293 0.686 rpy=1.5708 0 0, axis 0 -1 0, limit lower=-1.5 upper=1.5 effort=0 velocity=0
- joint ManipulatorBaseFixed: origin xyz=0.157269945428792 0.0354609509421621 0.707041900761443 rpy=1.5707963267949 0 3.14159265358979 -> xyz=0.15727 0.035461 0.70704 rpy=1.5708 0 3.1416
- joint lwheel_centers_fixed: axis 0 1 0 -> 0 0 0
- joint rwheel_centers_fixed: axis 0 1 0 -> 0 0 0
