Commit message: Moveit! exps

File: software/ros/workspaces/master/src/valter/robots/valter_initial.URDF (robot description, URDF)
Before this commit: robot valter, 46 links, 45 joints
Joints:
- joint LForearmYawJoint: limit (none) -> lower=-0.1 upper=0.4 effort=0 velocity=0; type fixed -> revolute
- joint LHandPitchJoint: type fixed -> revolute
- joint LHandYawJoint: type fixed -> revolute
