Commit message: ROS: valter_moveit package added to working set of workspaces

File: software/ros/workspaces/master/src/valter/robots/valter.URDF (robot description, URDF)
Before this commit: robot valter, 46 links, 45 joints
Joints:
- removed joint Head Pitch
- removed joint Head Yaw
- removed joint Left Arm Joint
- removed joint Left Forearm Joint
- removed joint Left Limb Joint
- removed joint Left Shoulder Yaw
- removed joint Torso Pitch
- removed joint Trunk Yaw
- added joint HeadJoint: type revolute, parent Neck, child Head, origin xyz=0.0085 0.05 0 rpy=0 0 0, axis 0 0 -1, limit lower=0 upper=0.85 effort=0 velocity=0
- added joint LArmElbowJoint: type revolute, parent LArm, child LArmElbow, origin xyz=0 -0.39975 0 rpy=-1.5708 0 1.5708, axis 0 0 -1, limit lower=-0.9 upper=0.9 effort=0 velocity=0
- added joint LArmJoint: type revolute, parent LShoulder, child LArm, origin xyz=0 0.116 0 rpy=-3.1416 0 1.5708, axis 0 0 -1, limit lower=-1.5 upper=0 effort=0 velocity=0
- added joint LShoulderJoint: type revolute, parent LTorso, child LShoulder, origin xyz=0.1085 0.31956 0.067 rpy=1.5708 0 1.5708, axis 0 1 0, limit lower=-1.5 upper=0.5 effort=0 velocity=0
- added joint LTorsoJoint: type revolute, parent Torso, child LTorso, origin xyz=0.10841 0 -0.09 rpy=3.1416 0 -3.1416, axis 0 -1 0, limit lower=0 upper=0.85 effort=0 velocity=0
- added joint NeckJoint: type revolute, parent Torso, child Neck, origin xyz=-0.00017682 0.42056 0 rpy=0 0 0, axis 0 -1 0, limit lower=-1.57 upper=1.57 effort=0 velocity=0
- added joint TorsoJoint: type revolute, parent Trunk, child Torso, origin xyz=0 0.45 0 rpy=0 0 0, axis 0 0 -1, limit lower=0 upper=1 effort=0 velocity=0
- added joint TrunkJoint: type revolute, parent Base, child Trunk, origin xyz=-0.01423 0.00097293 0.686 rpy=1.5708 0 0, axis 0 -1 0, limit lower=-1.5 upper=1.5 effort=0 velocity=0

Commit message: Valter MoveIt! preparations for experiments

File: software/ros/workspaces/master/src/valter/robots/valter.URDF (robot description, URDF)
Before this commit: robot valter, 46 links, 45 joints
Links:
- link Base: mass 12.7723641606721 -> None
- link GripperL: mass 0.0398581317877607 -> None
- link GripperR: mass 0.0398581317877607 -> None
- link Head: mass 5.04298545454377 -> None
- link LArm: mass 0.244790015736888 -> None
- link LArmElbow: mass 0.0397123450849927 -> None
- link LFinger0: mass 0.02336143148626 -> None
- link LFinger1: mass 0.02336143148626 -> None
- link LFinger2: mass 0.02336143148626 -> None
- link LFinger3: mass 0.02336143148626 -> None
- link LFinger4: mass 0.02336143148626 -> None
- link LFinger5: mass 0.02336143148626 -> None
- link LForearmRoll: mass 0.93501476271025 -> None
- link LForearmYaw: mass 0.60265 -> None
- link LHandPitch: mass 0.0061941814843542 -> None
- link LHandYaw: mass 0.312277803709901 -> None
- link LShoulder: mass 0.175328671502516 -> None
- link LTorso: mass 7.0955682087774 -> None
- link LWheel: mass 3.62031355964479 -> None
- link ManipulatorBase: mass 0.178834143520891 -> None
- link ManipulatorLink1: mass 0.478012742893284 -> None
- link ManipulatorLink2: mass 0.304515245459477 -> None
- link ManipulatorLink3: mass 0.227882111375496 -> None
- link ManipulatorLink4: mass 0.42934890554545 -> None
- link Neck: mass 0.264426936484469 -> None
- link RArm: mass 0.244790015736889 -> None
- link RArmElbow: mass 0.0397123450849928 -> None
- link RFinger0: mass 0.02336143148626 -> None
- link RFinger1: mass 0.02336143148626 -> None
- link RFinger2: mass 0.02336143148626 -> None
- link RFinger3: mass 0.02336143148626 -> None
- link RFinger4: mass 0.02336143148626 -> None
- link RFinger5: mass 0.0233614314862599 -> None
- link RForearmRoll: mass 0.935014762710249 -> None
- link RForearmYaw: mass 0.60265 -> None
- link RHandPitch: mass 0.00619418148435421 -> None
- link RHandYaw: mass 0.312277803709901 -> None
- link RShoulder: mass 0.175328671502516 -> None
- link RTorso: mass 7.0955682087774 -> None
- link RWheel: mass 3.62031355964479 -> None
- link Torso: mass 12.3493829426964 -> None
- link Trunk: mass 27.438 -> None
- link lwheel_centers: mass 0.0783773140784395 -> None
- link rwheel_centers: mass 0.0783773140784392 -> None
- link support_wheels: mass 1.30791131979034 -> None
- link support_wheels_centers: mass 0.101015328916835 -> None

Commit message: MoveIt! experiments

File: software/ros/workspaces/master/src/valter/robots/valter.URDF (robot description, URDF)
Before this commit: robot valter, 46 links, 45 joints
Joints:
- joint LWheelJoint: type continuous -> fixed
- joint RForearmYawJoint: type revolute -> fixed
- joint RHandPitchJoint: type revolute -> fixed
- joint RHandYawJoint: type revolute -> fixed
- joint RWheelJoint: type continuous -> fixed

Commit message: active dev commit

File: software/ros/workspaces/master/src/valter/robots/valter.URDF (robot description, URDF)
Before this commit: robot valter, 46 links, 45 joints
Joints:
- joint LArmJoint: axis 0 0 -1 -> 0 0 1; limit lower=-1.5 upper=0 effort=0 velocity=0 -> lower=0 upper=1.5 effort=0 velocity=0

Commit message: Right Arm expclient <-> ROS

File: software/ros/workspaces/master/src/valter/robots/valter.URDF (robot description, URDF)
Before this commit: robot valter, 46 links, 45 joints
Joints:
- joint LArmElbowJoint: axis 0 0 -1 -> 0 0 1
- joint LShoulderJoint: axis 0 1 0 -> 0 -1 0; limit lower=-1.5 upper=0.5 effort=0 velocity=0 -> lower=-0.5 upper=1.5 effort=0 velocity=0

Commit message: ROS right Arm MoveIt config modifications

File: software/ros/workspaces/master/src/valter/robots/valter.URDF (robot description, URDF)
Before this commit: robot valter, 46 links, 45 joints
Joints:
- joint RArmElbowJoint: axis 0 0 -1 -> 0 0 1
- joint RShoulderJoint: axis 0 -1 0 -> 0 1 0; limit lower=-1.5 upper=0.5 effort=0 velocity=0 -> lower=-0.5 upper=1.5 effort=0 velocity=0

Commit message: Left and Right Torso Joint pos calibration

File: software/ros/workspaces/master/src/valter/robots/valter.URDF (robot description, URDF)
Before this commit: robot valter, 46 links, 45 joints
Joints:
- joint LTorsoJoint: limit lower=0 upper=0.85 effort=0 velocity=0 -> lower=0 upper=0.925 effort=0 velocity=0
- joint RTorsoJoint: axis 0 -1 0 -> 0 1 0; limit lower=-0.85 upper=0 effort=0 velocity=0 -> lower=0 upper=0.88 effort=0 velocity=0
